File: hardware/0.1.1/ecp5-mini.kicad_pcb (KiCad board)
At the start: 4 copper layers, 52 x 27 mm, 111 parts, among them J1 Micro_SD_Card, J2 JTAG, J3 S7 Mini, J4 S7 Mini, J5 USB_C_Receptacle_USB2.0, Q1 BSS138, Q2 BSS138, Q3 BSS138, Q4 BSS138, SW1 KMR2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

Commit message: Update board date and version
Other:
- board text added: "2020-12-09"
- board text added: "Rev 0.1.1"
- board text removed: "2020-09-13"
- board text removed: "Rev 0.1"
